File: Schematic/exed.kicad_sch (KiCad schematic)
At the start: 136 parts, among them J1 BananaPlus, J10 PLLDivider, J11 CounterControl, J12 CounterOutput, J13 PLLOutput, J14 PLLOutput, J15 LogicLow, J2 BananaMinus, J3 ShiftInput, J4 XOR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

Commit message: Changed footprint of electrolytic to smd 0603
Parts:
- C1, C11, C13, C16, C18, C2, C5, C6, C9: footprint Capacitor_THT:CP_Radial_D4.0mm_P2.00mm -> Capacitor_SMD:C_0603_1608Metric_Pad1.08x0.95mm_HandSolder
- C10, C3, C7: footprint Capacitor_SMD:C_1206_3216Metric_Pad1.33x1.80mm_HandSolder -> Capacitor_SMD:C_0603_1608Metric_Pad1.08x0.95mm_HandSolder
Changed lines of the file:
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@@
     (property "Reference" "C2" (id 0) (at 53.8861 81.28 90))
     (property "Value" "1u" (id 1) (at 53.8861 83.82 90))
-    (property "Footprint" "Capacitor_THT:CP_Radial_D4.0mm_P2.00mm" (id 2) (at 53.34 87.63 0)
+    (property "Footprint" "Capacitor_SMD:C_0603_1608Metric_Pad1.08x0.95mm_HandSolder" (id 2) (at 53.34 87.63 0)
       (effects (font (size 1.27 1.27)) hide)
     )
@@
     (property "Reference" "C5" (id 0) (at 70.5739 185.42 90))
     (property "Value" "1u" (id 1) (at 70.5739 187.96 90))
-    (property "Footprint" "Capacitor_THT:CP_Radial_D4.0mm_P2.00mm" (id 2) (at 71.12 191.77 0)
+    (property "Footprint" "Capacitor_SMD:C_0603_1608Metric_Pad1.08x0.95mm_HandSolder" (id 2) (at 71.12 191.77 0)
       (effects (font (size 1.27 1.27)) hide)
     )
@@
     (property "Reference" "C16" (id 0) (at 213.36 110.49 90))
     (property "Value" "1u" (id 1) (at 208.28 110.49 90))
-    (property "Footprint" "Capacitor_THT:CP_Radial_D4.0mm_P2.00mm" (id 2) (at 210.82 109.22 0)
+    (property "Footprint" "Capacitor_SMD:C_0603_1608Metric_Pad1.08x0.95mm_HandSolder" (id 2) (at 210.82 109.22 0)
       (effects (font (size 1.27 1.27)) hide)
     )
@@
     (property "Reference" "C18" (id 0) (at 268.6939 20.32 90))
     (property "Value" "1u" (id 1) (at 268.6939 22.86 90))
-    (property "Footprint" "Capacitor_THT:CP_Radial_D4.0mm_P2.00mm" (id 2) (at 269.24 26.67 0)
+    (property "Footprint" "Capacitor_SMD:C_0603_1608Metric_Pad1.08x0.95mm_HandSolder" (id 2) (at 269.24 26.67 0)
       (effects (font (size 1.27 1.27)) hide)
     )
@@
     (property "Reference" "C13" (id 0) (at 148.0439 119.38 90))
     (property "Value" "1u" (id 1) (at 148.0439 121.92 90))
-    (property "Footprint" "Capacitor_THT:CP_Radial_D4.0mm_P2.00mm" (id 2) (at 148.59 125.73 0)
+    (property "Footprint" "Capacitor_SMD:C_0603_1608Metric_Pad1.08x0.95mm_HandSolder" (id 2) (at 148.59 125.73 0)
       (effects (font (size 1.27 1.27)) hide)
     )
@@
     (property "Reference" "C7" (id 0) (at 82.5436 86.36 90))
     (property "Value" "10n" (id 1) (at 82.5436 83.82 90))
-    (property "Footprint" "Capacitor_SMD:C_1206_3216Metric_Pad1.33x1.80mm_HandSolder" (id 2) (at 82.55 80.01 0)
+    (property "Footprint" "Capacitor_SMD:C_0603_1608Metric_Pad1.08x0.95mm_HandSolder" (id 2) (at 82.55 80.01 0)
       (effects (font (size 1.27 1.27)) hide)
     )
@@
     (property "Reference" "C11" (id 0) (at 134.62 86.36 90))
     (property "Value" "1u" (id 1) (at 134.62 83.82 90))
-    (property "Footprint" "Capacitor_THT:CP_Radial_D4.0mm_P2.00mm" (id 2) (at 134.62 80.01 0)
+    (property "Footprint" "Capacitor_SMD:C_0603_1608Metric_Pad1.08x0.95mm_HandSolder" (id 2) (at 134.62 80.01 0)
       (effects (font (size 1.27 1.27)) hide)
     )
@@
     (property "Reference" "C9" (id 0) (at 100.8761 39.37 90))
     (property "Value" "1u" (id 1) (at 100.8761 41.91 90))
-    (property "Footprint" "Capacitor_THT:CP_Radial_D4.0mm_P2.00mm" (id 2) (at 100.33 45.72 0)
+    (property "Footprint" "Capacitor_SMD:C_0603_1608Metric_Pad1.08x0.95mm_HandSolder" (id 2) (at 100.33 45.72 0)
       (effects (font (size 1.27 1.27)) hide)
     )
@@
     (property "Reference" "C3" (id 0) (at 64.7637 86.36 90))
     (property "Value" "10n" (id 1) (at 64.7637 83.82 90))
-    (property "Footprint" "Capacitor_SMD:C_1206_3216Metric_Pad1.33x1.80mm_HandSolder" (id 2) (at 64.77 80.01 0)
+    (property "Footprint" "Capacitor_SMD:C_0603_1608Metric_Pad1.08x0.95mm_HandSolder" (id 2) (at 64.77 80.01 0)
       (effects (font (size 1.27 1.27)) hide)
     )
@@
     (property "Reference" "C10" (id 0) (at 116.8337 86.36 90))
     (property "Value" "10n" (id 1) (at 116.8337 83.82 90))
-    (property "Footprint" "Capacitor_SMD:C_1206_3216Metric_Pad1.33x1.80mm_HandSolder" (id 2) (at 116.84 80.01 0)
+    (property "Footprint" "Capacitor_SMD:C_0603_1608Metric_Pad1.08x0.95mm_HandSolder" (id 2) (at 116.84 80.01 0)
       (effects (font (size 1.27 1.27)) hide)
     )
@@
       (effects (font (size 1.27 1.27)) (justify left))
     )
-    (property "Footprint" "Capacitor_THT:CP_Radial_D4.0mm_P2.00mm" (id 2) (at 53.34 29.21 0)
+    (property "Footprint" "Capacitor_SMD:C_0603_1608Metric_Pad1.08x0.95mm_HandSolder" (id 2) (at 53.34 29.21 0)
       (effects (font (size 1.27 1.27)) hide)
     )
@@
       (effects (font (size 1.27 1.27)) (justify left))
     )
-    (property "Footprint" "Capacitor_THT:CP_Radial_D4.0mm_P2.00mm" (id 2) (at 76.2 27.94 0)
+    (property "Footprint" "Capacitor_SMD:C_0603_1608Metric_Pad1.08x0.95mm_HandSolder" (id 2) (at 76.2 27.94 0)
       (effects (font (size 1.27 1.27)) hide)
     )
@@
     )
     (path "/f290457b-9f97-4d03-807e-706611da0cd7"
-      (reference "C1") (unit 1) (value "1u") (footprint "Capacitor_THT:CP_Radial_D4.0mm_P2.00mm")
+      (reference "C1") (unit 1) (value "1u") (footprint "Capacitor_SMD:C_0603_1608Metric_Pad1.08x0.95mm_HandSolder")
     )
     (path "/21a9ebd0-2e13-4f04-937b-e0786bd700b5"
-      (reference "C2") (unit 1) (value "1u") (footprint "Capacitor_THT:CP_Radial_D4.0mm_P2.00mm")
+      (reference "C2") (unit 1) (value "1u") (footprint "Capacitor_SMD:C_0603_1608Metric_Pad1.08x0.95mm_HandSolder")
     )
     (path "/bee73ae4-300b-4adb-a65c-6f5f9033b4eb"
-      (reference "C3") (unit 1) (value "10n") (footprint "Capacitor_SMD:C_1206_3216Metric_Pad1.33x1.80mm_HandSolder")
+      (reference "C3") (unit 1) (value "10n") (footprint "Capacitor_SMD:C_0603_1608Metric_Pad1.08x0.95mm_HandSolder")
     )
     (path "/514746e1-0ad2-4622-a8a2-879123c2235f"
@@
     )
     (path "/47b4086f-c2c0-4653-8e7e-650349a72da9"
-      (reference "C5") (unit 1) (value "1u") (footprint "Capacitor_THT:CP_Radial_D4.0mm_P2.00mm")
+      (reference "C5") (unit 1) (value "1u") (footprint "Capacitor_SMD:C_0603_1608Metric_Pad1.08x0.95mm_HandSolder")
     )
     (path "/feeacc79-c112-4cbf-8876-bee11e4d5353"
-      (reference "C6") (unit 1) (value "1u") (footprint "Capacitor_THT:CP_Radial_D4.0mm_P2.00mm")
+      (reference "C6") (unit 1) (value "1u") (footprint "Capacitor_SMD:C_0603_1608Metric_Pad1.08x0.95mm_HandSolder")
     )
     (path "/92942b14-44e1-4def-be1c-cedf069d0b6a"
-      (reference "C7") (unit 1) (value "10n") (footprint "Capacitor_SMD:C_1206_3216Metric_Pad1.33x1.80mm_HandSolder")
+      (reference "C7") (unit 1) (value "10n") (footprint "Capacitor_SMD:C_0603_1608Metric_Pad1.08x0.95mm_HandSolder")
     )
     (path "/d16db643-0edf-4407-87be-4cfc9d8420ac"
@@
     )
     (path "/a324955d-3bd0-49cb-92be-0ae869281102"
-      (reference "C9") (unit 1) (value "1u") (footprint "Capacitor_THT:CP_Radial_D4.0mm_P2.00mm")
+      (reference "C9") (unit 1) (value "1u") (footprint "Capacitor_SMD:C_0603_1608Metric_Pad1.08x0.95mm_HandSolder")
     )
     (path "/bf3fb57c-237e-4444-af32-ff4404e8918b"
-      (reference "C10") (unit 1) (value "10n") (footprint "Capacitor_SMD:C_1206_3216Metric_Pad1.33x1.80mm_HandSolder")
+      (reference "C10") (unit 1) (value "10n") (footprint "Capacitor_SMD:C_0603_1608Metric_Pad1.08x0.95mm_HandSolder")
     )
     (path "/99063560-a490-473d-bb51-3974a708339e"
-      (reference "C11") (unit 1) (value "1u") (footprint "Capacitor_THT:CP_Radial_D4.0mm_P2.00mm")
+      (reference "C11") (unit 1) (value "1u") (footprint "Capacitor_SMD:C_0603_1608Metric_Pad1.08x0.95mm_HandSolder")
     )
     (path "/200e8f3f-6af4-48da-aa53-95baf026fc74"
@@
     )
     (path "/69d4cd1f-7360-4307-babb-8c43e8e2211f"
-      (reference "C13") (unit 1) (value "1u") (footprint "Capacitor_THT:CP_Radial_D4.0mm_P2.00mm")
+      (reference "C13") (unit 1) (value "1u") (footprint "Capacitor_SMD:C_0603_1608Metric_Pad1.08x0.95mm_HandSolder")
     )
     (path "/9ff3b2a6-c2f0-4b4a-bb8c-5524f748a597"
@@
     )
     (path "/55b6b8d1-9d52-4a9b-9277-ac4e8cae0a22"
-      (reference "C16") (unit 1) (value "1u") (footprint "Capacitor_THT:CP_Radial_D4.0mm_P2.00mm")
+      (reference "C16") (unit 1) (value "1u") (footprint "Capacitor_SMD:C_0603_1608Metric_Pad1.08x0.95mm_HandSolder")
     )
     (path "/e57b4110-4a43-4f92-9afd-69d660ddeab7"
@@
     )
     (path "/619b10af-6e29-4329-8e71-ad0a0e12fd90"
-      (reference "C18") (unit 1) (value "1u") (footprint "Capacitor_THT:CP_Radial_D4.0mm_P2.00mm")
+      (reference "C18") (unit 1) (value "1u") (footprint "Capacitor_SMD:C_0603_1608Metric_Pad1.08x0.95mm_HandSolder")
     )
     (path "/f3bb0716-57f4-40d2-8083-041c44ef84c2"

Commit message: Final version v0.1
Parts:
- removed R37: 10M, Resistor_SMD:R_0603_1608Metric_Pad0.98x0.95mm_HandSolder, symbol Device:R_Small
- R3: value 500 -> 330
Connections:
- net at J10.1 (Pin_1), R39.2, U7.14 (SigIn): now also J10.2 (Pin_2); no longer J9.1 (Pin_1)
- net at J9.2 (Pin_2), R40.2, U7.3 (RefIn): now also J9.1 (Pin_1); no longer J10.2 (Pin_2)
